Commit message: push env changed

File: pybullet_robot_envs/robot_data/kuka_kr6_support/urdf/kr6r700sixx_copy.urdf (robot description, URDF)
Before this commit: robot kuka_kr6r700, 11 links, 10 joints
Links:
- removed link leftfinger
- removed link rightfinger
- link link_4: mass 0.5 -> 1.0
- link link_5: mass 0.3 -> 1.0
- link link_6: mass 0.1 -> 1.0
- link tool0: mass 0.3 -> None; geometry collision box size=.03 .03 .2; visual mesh filename=../cube.obj scale=.03 .03 .2
Joints:
- removed joint finger_joint1
- removed joint finger_joint2
