Commit message: add reach_her env and push_her env and waiting for testing

File: pybullet_robot_envs/robot_data/kuka_kr6_support/urdf/kr6r700sixx.urdf (robot description, URDF)
Before this commit: robot kuka_kr6r700, 9 links, 8 joints
Links:
- link base: mass None -> 1.0
- link link_1: mass None -> 1.0
- link link_2: mass None -> 1.0
- link link_3: mass None -> 1.0
- link link_4: mass None -> 1.0
- link link_5: mass None -> 1.0
- link link_6: mass None -> 1.0
- link tool0: mass None -> 1.0

Commit message: add Pick task, but it failed

File: pybullet_robot_envs/robot_data/kuka_kr6_support/urdf/kr6r700sixx.urdf (robot description, URDF)
Before this commit: robot kuka_kr6r700, 11 links, 10 joints
Joints:
- joint finger_joint1: limit lower=0.0 upper=0.1 effort=20 velocity=0.2 -> lower=0.01 upper=0.1 effort=20 velocity=0.01
- joint finger_joint2: limit lower=0.0 upper=0.1 effort=20 velocity=0.2 -> lower=0.01 upper=0.1 effort=20 velocity=0.01
