Commit message: remove pandas envs

File: pybullet_robot_envs/robot_data/kuka_kr6_support/cube.urdf (robot description, URDF)
Before this commit: robot cube.urdf, 1 links, 0 joints
Links:
- link baseLink: geometry collision box size=.08 .08 .08; visual mesh filename=cube.obj scale=.08 .08 .08

File: pybullet_robot_envs/robot_data/kuka_kr6_support/urdf/kr6r700sixx.urdf (robot description, URDF)
Before this commit: robot kuka_kr6r700, 11 links, 10 joints
Joints:
- joint finger_joint1: limit lower=0.0 upper=0.01 effort=20 velocity=0.2 -> lower=0.0 upper=0.1 effort=20 velocity=0.2
- joint finger_joint2: limit lower=0.0 upper=0.01 effort=20 velocity=0.2 -> lower=0.0 upper=0.1 effort=20 velocity=0.2
